Commit message: Make updates

File: catkin_ws/src/my_robot/urdf/my_robot.xacro (robot description, xacro)
@@ -2,4 +2,5 @@
 <robot name="my_robot"
     xmlns:xacro="http://www.ros.org/wiki/xacro">
+    <xacro:include filename="$(find my_robot)/urdf/my_robot.gazebo" />
     <link name="robot_footprint"></link>
     <joint name="robot_footprint_joint" type="fixed">
@@ -78,4 +79,5 @@
                 <cylinder radius="0.1" length="0.05"/>
             </geometry>
+            <material name="blue"/>
         </visual>
     </link>
@@ -102,4 +104,5 @@
                 <cylinder radius="0.1" length="0.05"/>
             </geometry>
+            <material name="blue"/>
         </visual>
     </link>
@@ -131,5 +134,5 @@
       />
         </inertial>
-        <visual>
+        <visual name="camera_visual">
             <origin xyz="0 0 0" rpy=" 0 0 0"/>
             <geometry>
@@ -137,5 +140,5 @@
             </geometry>
         </visual>
-        <collision>
+        <collision name="collision">
             <origin xyz="0 0 0" rpy=" 0 0 0"/>
             <geometry>
@@ -146,3 +149,38 @@
     <joint type="fixed" name="camera_joint">
         <origin xyz="0.2 0 0" rpy="0 0 0"/>
-    </robot>
+        <child link="camera"/>
+        <parent link="chassis"/>
+        <axis xyz="0 1 0" rpy="0 0 0"/>
+        <limit effort="10000" velocity="1000"/>
+        <dynamics damping="1.0" friction="1.0"/>
+    </joint>
+    <link name="hokuyo">
+        <inertial>
+            <mass value="1e-5"/>
+            <origin xyz="0 0 0" rpy="0 0 0"/>
+            <inertia
+            ixx="1e-6" ixy="0" ixz="0" iyy="1e-6" iyz="0" izz="1e-6"
+            />
+        </inertial>
+        <collision name='collision'>
+            <origin xyz="0 0 0" rpy=" 0 0 0"/>
+            <geometry>
+                <box size="0.1 0.1 0.1"/>
+            </geometry>
+        </collision>
+        <visual name='hokuyo_visual'>
+            <origin xyz="0 0 0" rpy="0 0 0"/>
+            <geometry>
+                <mesh filename="package://my_robot/meshes/hokuyo.dae"/>
+            </geometry>
+        </visual>
+    </link>
+    <joint type="fixed" name="hokuyo_joint">
+        <origin xyz="0.15 0.0 0.1" rpy="0 0 0"/>
+        <child link="hokuyo"/>
+        <parent link="chassis"/>
+        <axis xyz="0 1 0" rpy="0 0 0"/>
+        <limit effort="10000" velocity="1000"/>
+        <dynamics damping="1.0" friction="1.0"/>
+    </joint>
+</robot>
